File: stm32_minimal_dev.kicad_sch (KiCad schematic)
At the start: 32 parts, among them J1 Conn_01x12_Male, J2 Conn_01x12_Male, J3 Conn_01x08_Male, J4 USB_B_Micro, SW1 SW_SPDT, U1 AMS1117-3.3, U2 STM32F103C8T6, Y1 16MHz

Commit message: updated files
Connections:
- net GND: now also J4.5
- no-connect marks 8 -> 7
Changed lines of the file:
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@@
   (no_connect (at 35.56 76.2))
   (no_connect (at 35.56 73.66))
-  (no_connect (at 260.35 119.38))
   (no_connect (at 260.35 116.84))
   (no_connect (at 35.56 71.12))
@@
     (pin "1")
     (pin "2")
+  )
+  (symbol (lib_id "power:GND") (at 260.35 119.38 0) (unit 1)
+    (in_bom yes) (on_board yes) (fields_autoplaced)
+    (property "Reference" "#PWR0105" (id 0) (at 260.35 125.73 0)
+      (effects (font (size 1.27 1.27)) hide)
+    )
+    (property "Value" "GND" (id 1) (at 260.35 124.46 0))
+    (property "Footprint" "" (id 2) (at 260.35 119.38 0)
+      (effects (font (size 1.27 1.27)) hide)
+    )
+    (property "Datasheet" "" (id 3) (at 260.35 119.38 0)
+      (effects (font (size 1.27 1.27)) hide)
+    )
+    (pin "1")
   )
   (symbol (lib_id "Mechanical:MountingHole") (at 34.29 156.21 0) (unit 1)
@@
       (reference "#PWR0104") (unit 1) (value "GND") (footprint "")
     )
+    (path "/62ff518b-de58-45da-85d3-d0cddcde2e8c"
+      (reference "#PWR0105") (unit 1) (value "GND") (footprint "")
+    )
     (path "/f62969ba-6653-4089-b38e-8c0ef2fba9df"
